File: CAD/XMICRO-MEMORY.sch (EAGLE design)
At the start: 72 parts, among them Q1 2N4403, U1 28C256, U10 74244, U11 74138, U12 74138, U13 74244, U14 74244, U15 74244, U16 74245, U2 AS6C4008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

Commit message: Updated schematic xrefs to indicate signal direction.
Other:
- note removed: "ADDRESS BUS"
- note removed: "DATA BUS"
- moved on the sheet: U6A, U8F
